Commit message: 更新 sentry.urdf.xacro 文件，修改多个链接和关节的颜色、尺寸及位置，优化机器人模型的视觉表现

File: src/spr_sentry_description/sentry.urdf.xacro (robot description, xacro)
@@ -6,5 +6,5 @@
       <origin xyz="0 0 0" rpy="0 0 0" />
       <material name="">
-        <color rgba="0.752941176470588 0.752941176470588 0.752941176470588 1" />
+        <color rgba="1 0 0 1" />
       </material>
       <geometry>
@@ -20,5 +20,5 @@
   </link>
   <joint name="base_joint" type="fixed">
-    <origin xyz="0 0 0.0" rpy="0 0 0" />
+    <origin xyz="0 0 0.15" rpy="0 0 0" />
     <parent link="odom" />
     <child link="base_link" />
@@ -29,8 +29,8 @@
       <origin xyz="0 0 0" rpy="0 0 0" />
       <material name="">
-        <color rgba="0.792156862745098 0.819607843137255 0.933333333333333 1" />
+        <color rgba="0 1 1 1" />
       </material>
       <geometry>
-        <cylinder radius="0.1" length="0.1" />
+        <cylinder radius="0.2" length="0.1" />
       </geometry>
     </visual>
@@ -38,10 +38,10 @@
       <origin xyz="0 0 0" rpy="0 0 0" />
       <geometry>
-        <cylinder radius="0.1" length="0.1" />
+        <cylinder radius="0.2" length="0.1" />
       </geometry>
     </collision>
   </link>
   <joint name="bigyaw_joint" type="continuous">
-      <origin xyz="0 0 0.0" rpy="0 0 0" />
+      <origin xyz="0 0 0.1" rpy="0 0 0" />
       <parent link="base_link" />
       <child link="bigyaw_link" />
@@ -52,5 +52,51 @@
       <origin xyz="0 0 0" rpy="0 0 0" />
       <material name="">
-        <color rgba="0.792156862745098 0.819607843137255 0.933333333333333 1" />
+        <color rgba="0 0 1 1" />
+      </material>
+      <geometry>
+        <cylinder radius="0.03" length="0.3" />
+      </geometry>
+    </visual>
+    <collision>
+      <origin xyz="0 0 0" rpy="0 0 0" />
+      <geometry>
+        <cylinder radius="0.03" length="0.3" />
+      </geometry>
+    </collision>
+  </link>
+  <joint name="small_yaw_joint" type="continuous">
+    <origin xyz="0 0 0.1" rpy="0 0 0" />
+    <parent link="bigyaw_link" />
+    <child link="small_yaw_link" />
+    <axis xyz="0 0 1" />
+  </joint>
+  <link name="pitch_link">
+    <visual>
+      <origin xyz="0.14 0 0" rpy="0 1.5708 0" />
+      <material name="">
+        <color rgba="0 1 1 1" />
+      </material>
+      <geometry>
+        <cylinder radius="0.05" length="0.28" />
+      </geometry>
+    </visual>
+    <collision>
+      <origin xyz="0.14 0 0" rpy="0 1.5708 0" />
+      <geometry>
+        <cylinder radius="0.05" length="0.28" />
+      </geometry>
+    </collision>
+  </link>
+  <joint name="pitch_joint" type="continuous">
+    <origin xyz="0 0 0.15" rpy="0 0 0" />
+    <parent link="small_yaw_link" />
+    <child link="pitch_link" />
+    <axis xyz="0 1 0" />
+  </joint>
+  <link name="left_wheel_front_link">
+    <visual>
+      <origin xyz="0 0 0" rpy="1.5708 0 0" />
+      <material name="">
+        <color rgba="1 1 0 1" />
       </material>
       <geometry>
@@ -59,5 +105,5 @@
     </visual>
     <collision>
-      <origin xyz="0 0 0" rpy="0 0 0" />
+      <origin xyz="0 0 0" rpy="1.5708 0 0" />
       <geometry>
         <cylinder radius="0.1" length="0.1" />
@@ -65,15 +111,15 @@
     </collision>
   </link>
-  <joint name="small_yaw_joint" type="continuous">
-    <origin xyz="0 0 0.0" rpy="0 0 0" />
-    <parent link="bigyaw_link" />
-    <child link="small_yaw_link" />
-    <axis xyz="0 0 1" />
+  <joint name="left_wheel_front_joint" type="continuous">
+    <origin xyz="-0.2 0.25 -0.05" rpy="0 0 0" />
+    <parent link="base_link" />
+    <child link="left_wheel_front_link" />
+    <axis xyz="0 1 0" />
   </joint>
-  <link name="pitch_link">
+  <link name="right_wheel_front_link">
     <visual>
-      <origin xyz="0 0 0" rpy="0 0 0" />
+      <origin xyz="0 0 0" rpy="1.5708 0 0" />
       <material name="">
-        <color rgba="0.792156862745098 0.819607843137255 0.933333333333333 1" />
+        <color rgba="1 1 0 1" />
       </material>
       <geometry>
@@ -82,5 +128,5 @@
     </visual>
     <collision>
-      <origin xyz="0 0 0" rpy="0 0 0" />
+      <origin xyz="0 0 0" rpy="1.5708 0 0" />
       <geometry>
         <cylinder radius="0.1" length="0.1" />
@@ -88,15 +134,15 @@
     </collision>
   </link>
-  <joint name="pitch_joint" type="continuous">
-    <origin xyz="0 0 0.0" rpy="0 0 0" />
-    <parent link="small_yaw_link" />
-    <child link="pitch_link" />
+  <joint name="right_wheel_front_joint" type="continuous">
+    <origin xyz="-0.2 -0.25 -0.05" rpy="0 0 0" />
+    <parent link="base_link" />
+    <child link="right_wheel_front_link" />
     <axis xyz="0 1 0" />
   </joint>
-  <link name="left_wheel_front_link">
+  <link name="left_wheel_back_link">
     <visual>
-      <origin xyz="0 0 0" rpy="0 0 0" />
+      <origin xyz="0 0 0" rpy="1.5708 0 0" />
       <material name="">
-        <color rgba="0.792156862745098 0.819607843137255 0.933333333333333 1" />
+        <color rgba="1 1 0 1" />
       </material>
       <geometry>
@@ -105,51 +151,5 @@
     </visual>
     <collision>
-      <origin xyz="0 0 0" rpy="0 0 0" />
-      <geometry>
-        <cylinder radius="0.1" length="0.1" />
-      </geometry>
-    </collision>
-  </link>
-  <joint name="left_wheel_front_joint" type="continuous">
-    <origin xyz="0 0 0.0" rpy="0 0 0" />
-    <parent link="base_link" />
-    <child link="left_wheel_front_link" />
-    <axis xyz="0 1 0" />
-  </joint>
-  <link name="right_wheel_front_link">
-    <visual>
-      <origin xyz="0 0 0" rpy="0 0 0" />
-      <material name="">
-        <color rgba="0.792156862745098 0.819607843137255 0.933333333333333 1" />
-      </material>
-      <geometry>
-        <cylinder radius="0.1" length="0.1" />
-      </geometry>
-    </visual>
-    <collision>
-      <origin xyz="0 0 0" rpy="0 0 0" />
-      <geometry>
-        <cylinder radius="0.1" length="0.1" />
-      </geometry>
-    </collision>
-  </link>
-  <joint name="right_wheel_front_joint" type="continuous">
-    <origin xyz="0 0 0.0" rpy="0 0 0" />
-    <parent link="base_link" />
-    <child link="right_wheel_front_link" />
-    <axis xyz="0 1 0" />
-  </joint>
-  <link name="left_wheel_back_link">
-    <visual>
-      <origin xyz="0 0 0" rpy="0 0 0" />
-      <material name="">
-        <color rgba="0.792156862745098 0.819607843137255 0.933333333333333 1" />
-      </material>
-      <geometry>
-        <cylinder radius="0.1" length="0.1" />
-      </geometry>
-    </visual>
-    <collision>
-      <origin xyz="0 0 0" rpy="0 0 0" />
+      <origin xyz="0 0 0" rpy="1.5708 0 0" />
       <geometry>
         <cylinder radius="0.1" length="0.1" />
@@ -158,5 +158,5 @@
     </link>
     <joint name="left_wheel_back_joint" type="continuous">
-      <origin xyz="0 0 0.0" rpy="0 0 0" />
+      <origin xyz="0.2 0.25 -0.05" rpy="0 0 0" />
       <parent link="base_link" />
       <child link="left_wheel_back_link" />
@@ -165,7 +165,7 @@
     <link name="right_wheel_back_link">
         <visual>
-            <origin xyz="0 0 0" rpy="0 0 0" />
+            <origin xyz="0 0 0" rpy="1.5708 0 0" />
             <material name="">
-            <color rgba="0.792156862745098 0.819607843137255 0.933333333333333 1" />
+            <color rgba="1 1 0 1" />
             </material>
             <geometry>
@@ -174,5 +174,5 @@
         </visual>
         <collision>
-            <origin xyz="0 0 0" rpy="0 0 0" />
+            <origin xyz="0 0 0" rpy="1.5708 0 0" />
             <geometry>
                 <cylinder radius="0.1" length="0.1" />
@@ -181,5 +181,5 @@
     </link>
     <joint name="right_wheel_back_joint" type="continuous">
-        <origin xyz="0 0 0.0" rpy="0 0 0" />
+        <origin xyz="0.2 -0.25 -0.05" rpy="0 0 0" />
         <parent link="base_link" />
         <child link="right_wheel_back_link" />

Commit message: 调整云台 TF：上移 small_yaw 使 pitch 连接点位于其末端；新增 gimbal_controller 控制器包

File: src/spr_sentry_description/sentry.urdf.xacro (robot description, xacro)
@@ -50,5 +50,5 @@
   <link name="small_yaw_link">
     <visual>
-      <origin xyz="0 0 0" rpy="0 0 0" />
+      <origin xyz="0 0 0.1" rpy="0 0 0" />
       <material name="">
         <color rgba="0 0 1 1" />
@@ -89,5 +89,5 @@
   </link>
   <joint name="pitch_joint" type="continuous">
-    <origin xyz="0 0 0.15" rpy="0 0 0" />
+    <origin xyz="0 0 0.25" rpy="0 0 0" />
     <parent link="small_yaw_link" />
     <child link="pitch_link" />
