Commit message: 添加 gimbal_controller 生命周期函数，重构 gimbal_cmd 和 gimbal_state 消息，更新 PID 参数，添加不同模式下的控制函数

File: src/spr_ctrl_bring_up/description/sentry.xacro (robot description, xacro)
@@ -25,5 +25,5 @@
         VIRTUAL_JOINT,
     } Motor_Type_e;-->
-        <joint name="bigyaw_joint">
+        <joint name="big_yaw_joint">
             <param name="motor_name" value="bigyaw_motor" />
             <param name="can_bus" value="can0" />

Commit message: 实现云台串级PID控制与达妙MIT协议： - 硬件层新增 effort 命令接口，按电机类型打包(DJI int16 电流帧/DM MIT float 力矩帧) - 实现达妙 MIT 编解码(float_to_uint/uint_to_float、控制帧/回传帧解析)与使能帧 - 新增 EffortMockSystem 模拟硬件支持无真机调试 effort 链路 - gimbal_controller 接入位置环PID→effort 输出，发布 gimbal_state 状态 - 配置:云台关节接口调整、PID输出限幅、DM 映射满量程参数

File: src/spr_ctrl_bring_up/description/sentry.xacro (robot description, xacro)
@@ -5,9 +5,10 @@
         <!-- <hardware>
             <plugin>spr_hw_interface/SprHardwareInterface</plugin>
-            <param name="can_device_count_" value="2" />
+            <param name="can_device_count_">2</param>
          </hardware> -->
         <hardware>
-            <plugin>mock_components/GenericSystem</plugin>
-            <param name="calculate_dynamics">true</param>
+            <!-- 无真机时用 effort 模拟硬件调试位置环->effort 链路 -->
+            <plugin>spr_hw_interface/EffortMockSystem</plugin>
+            <param name="accel_per_effort">0.5</param>
         </hardware>
 <!--
@@ -30,69 +31,79 @@
     } Motor_Type_e;-->
         <joint name="big_yaw_joint">
-            <param name="motor_name" value="bigyaw_motor" />
-            <param name="can_bus" value="can0" />
-            <param name="tx_id" value="1" />
-            <param name="offset" value="0" />
-            <param name="motor_type" value="DM6006" />
+            <param name="motor_name">bigyaw_motor</param>
+            <param name="can_bus">can0</param>
+            <param name="tx_id">1</param>
+            <param name="offset">0</param>
+            <param name="motor_type">DM6006</param>
+            <param name="pos_max">12.5</param>
+            <param name="vel_max">30</param>
+            <param name="tor_max">10</param>
             <command_interface name="position" />
             <command_interface name="velocity" />
+            <command_interface name="effort" />
             <state_interface name="position" />
             <state_interface name="velocity" />
+            <state_interface name="effort" />
         </joint>
         <joint name="small_yaw_joint">
-            <param name="motor_name" value="small_yaw_motor" />
-            <param name="can_bus" value="can0" />
-            <param name="tx_id" value="2" />
-            <param name="offset" value="0" />
-            <param name="motor_type" value="GM6020" />
+            <param name="motor_name">small_yaw_motor</param>
+            <param name="can_bus">can0</param>
+            <param name="tx_id">2</param>
+            <param name="offset">0</param>
+            <param name="motor_type">GM6020</param>
+            <command_interface name="effort" />
+            <state_interface name="position" />
+            <state_interface name="velocity" />
+            <state_interface name="effort" />
+        </joint>
+        <joint name="pitch_joint">
+            <param name="motor_name">pitch_motor</param>
+            <param name="can_bus">can0</param>
+            <param name="tx_id">3</param>
+            <param name="offset">0</param>
+            <param name="motor_type">DM4310</param>
+            <param name="pos_max">12.5</param>
+            <param name="vel_max">30</param>
+            <param name="tor_max">10</param>
             <command_interface name="position" />
             <command_interface name="velocity" />
+            <command_interface name="effort" />
             <state_interface name="position" />
             <state_interface name="velocity" />
-        </joint>
-        <joint name="pitch_joint">
-            <param name="motor_name" value="pitch_motor" />
-            <param name="can_bus" value="can0" />
-            <param name="tx_id" value="3" />
-            <param name="offset" value="0" />
-            <param name="motor_type" value="DM4310" />
-            <command_interface name="position" />
-            <command_interface name="velocity" />
-            <state_interface name="position" />
-            <state_interface name="velocity" />
+            <state_interface name="effort" />
         </joint>
         <joint name="left_wheel_front_joint">
-            <param name="motor_name" value="left_wheel_front_motor" />
-            <param name="can_bus" value="can1" />
-            <param name="tx_id" value="1" />
-            <param name="offset" value="0" />
-            <param name="motor_type" value="M3508" />
+            <param name="motor_name">left_wheel_front_motor</param>
+            <param name="can_bus">can1</param>
+            <param name="tx_id">1</param>
+            <param name="offset">0</param>
+            <param name="motor_type">M3508</param>
             <command_interface name="velocity" />
             <state_interface name="velocity" />
         </joint>
         <joint name="right_wheel_front_joint">
-            <param name="motor_name" value="right_wheel_front_motor" />
-            <param name="can_bus" value="can1" />
-            <param name="tx_id" value="2" />
-            <param name="offset" value="0" />
-            <param name="motor_type" value="M3508" />
+            <param name="motor_name">right_wheel_front_motor</param>
+            <param name="can_bus">can1</param>
+            <param name="tx_id">2</param>
+            <param name="offset">0</param>
+            <param name="motor_type">M3508</param>
             <command_interface name="velocity" />
             <state_interface name="velocity" />
         </joint>
         <joint name="left_wheel_back_joint">
-            <param name="motor_name" value="left_wheel_back_motor" />
-            <param name="can_bus" value="can1" />
-            <param name="tx_id" value="3" />
-            <param name="offset" value="0" />
-            <param name="motor_type" value="M3508" />
+            <param name="motor_name">left_wheel_back_motor</param>
+            <param name="can_bus">can1</param>
+            <param name="tx_id">3</param>
+            <param name="offset">0</param>
+            <param name="motor_type">M3508</param>
             <command_interface name="velocity" />
             <state_interface name="velocity" />
         </joint>
         <joint name="right_wheel_back_joint">
-            <param name="motor_name" value="right_wheel_back_motor" />
-            <param name="can_bus" value="can1" />
-            <param name="tx_id" value="4" />
-            <param name="offset" value="0" />
-            <param name="motor_type" value="M3508" />
+            <param name="motor_name">right_wheel_back_motor</param>
+            <param name="can_bus">can1</param>
+            <param name="tx_id">4</param>
+            <param name="offset">0</param>
+            <param name="motor_type">M3508</param>
             <command_interface name="velocity" />
             <state_interface name="velocity" />

Commit message: 添加底盘控制器和遥控功能，更新相关配置文件，修正云台关节名称，新增 RViz 配置文件

File: src/spr_ctrl_bring_up/description/sentry.xacro (robot description, xacro)
@@ -30,5 +30,5 @@
         VIRTUAL_JOINT,
     } Motor_Type_e;-->
-        <joint name="big_yaw_joint">
+        <joint name="bigyaw_joint">
             <param name="motor_name">bigyaw_motor</param>
             <param name="can_bus">can0</param>
@@ -80,5 +80,6 @@
             <param name="offset">0</param>
             <param name="motor_type">M3508</param>
-            <command_interface name="velocity" />
+            <command_interface name="effort" />
+            <state_interface name="position" />
             <state_interface name="velocity" />
         </joint>
@@ -89,5 +90,6 @@
             <param name="offset">0</param>
             <param name="motor_type">M3508</param>
-            <command_interface name="velocity" />
+            <command_interface name="effort" />
+            <state_interface name="position" />
             <state_interface name="velocity" />
         </joint>
@@ -98,5 +100,6 @@
             <param name="offset">0</param>
             <param name="motor_type">M3508</param>
-            <command_interface name="velocity" />
+            <command_interface name="effort" />
+            <state_interface name="position" />
             <state_interface name="velocity" />
         </joint>
@@ -107,5 +110,6 @@
             <param name="offset">0</param>
             <param name="motor_type">M3508</param>
-            <command_interface name="velocity" />
+            <command_interface name="effort" />
+            <state_interface name="position" />
             <state_interface name="velocity" />
         </joint>

Commit message: 更新 README，添加 RViz 可视化调试说明；修改底盘控制器以支持里程计发布；优化 EffortMockSystem 参数；实现麦克纳姆轮正运动学与里程计更新功能

File: src/spr_ctrl_bring_up/description/sentry.xacro (robot description, xacro)
@@ -10,5 +10,6 @@
             <!-- 无真机时用 effort 模拟硬件调试位置环->effort 链路 -->
             <plugin>spr_hw_interface/EffortMockSystem</plugin>
-            <param name="accel_per_effort">0.5</param>
+            <param name="accel_per_effort">2</param>
+            <param name="max_velocity">50</param>
         </hardware>
 <!--

File: src/spr_sentry_description/sentry.urdf.xacro (robot description, xacro)
@@ -1,5 +1,5 @@
 <?xml version="1.0" encoding="utf-8"?>
 <robot name="sentry">
-  <link name="odom"/>
+  <link name="base_footprint"/>  <!-- 底盘里程计原点(URDF根)，odom->base_footprint 由 chassis_controller 动态发布 -->
   <link name="base_link">
     <visual>
@@ -21,5 +21,5 @@
   <joint name="base_joint" type="fixed">
     <origin xyz="0 0 0.15" rpy="0 0 0" />
-    <parent link="odom" />
+    <parent link="base_footprint" />
     <child link="base_link" />
     <axis xyz="0 0 0" />

Commit message: Refactor motor feedback decoding and chassis controller for Mecanum wheel layout
- Updated `spr_motor.cpp` to improve feedback decoding, including handling of position offsets and temperature readings.
- Modified `chassis_controller.cpp` to correct inverse kinematics calculations for Mecanum wheels, ensuring proper wheel direction and rotation semantics.
- Enhanced `chassis_controller_parameter.yaml` to include a parameter for wheel layout type, allowing for configuration of Mecanum wheel roller orientation.
- Adjusted `sentry_robot.xml` and `sentry.urdf.xacro` to correct the positions of the wheels and pitch link for accurate simulation.
- Introduced `dm_can_tool.py`, a new tool for real-time monitoring and control of DM motors via CAN, simplifying the debugging process.

File: src/spr_ctrl_bring_up/description/sentry.xacro (robot description, xacro)
@@ -53,10 +53,10 @@
             <param name="offset">0</param>
             <param name="motor_type">DM6006</param>
-            <param name="pos_max">12.5</param>
+            <param name="pos_max">3.14</param>
             <param name="vel_max">30</param>
             <param name="tor_max">10</param>
+            <command_interface name="effort" />
             <command_interface name="position" />
             <command_interface name="velocity" />
-            <command_interface name="effort" />
             <state_interface name="position" />
             <state_interface name="velocity" />
@@ -66,7 +66,10 @@
             <param name="motor_name">small_yaw_motor</param>
             <param name="can_bus">can0</param>
-            <param name="tx_id">6</param>
-            <param name="offset">0</param>
-            <param name="motor_type">GM6020</param>
+            <param name="tx_id">5</param>
+            <param name="offset">-1.805</param>
+            <param name="motor_type">DM4310</param>
+            <param name="pos_max">3.14</param>
+            <param name="vel_max">30</param>
+            <param name="tor_max">10</param>
             <command_interface name="effort" />
             <command_interface name="position"/>
@@ -78,13 +81,13 @@
             <param name="motor_name">pitch_motor</param>
             <param name="can_bus">can0</param>
-            <param name="tx_id">3</param>
-            <param name="offset">0</param>
+            <param name="tx_id">4</param>
+            <param name="offset">2.728</param>
             <param name="motor_type">DM4310</param>
-            <param name="pos_max">12.5</param>
+            <param name="pos_max">3.14</param>
             <param name="vel_max">30</param>
             <param name="tor_max">10</param>
+            <command_interface name="effort" />
             <command_interface name="position" />
             <command_interface name="velocity" />
-            <command_interface name="effort" />
             <state_interface name="position" />
             <state_interface name="velocity" />
@@ -97,5 +100,6 @@
             <param name="offset">0</param>
             <param name="motor_type">M3508</param>
-            <command_interface name="effort" />
+            <param name="reduction">19.2032</param>
+            <param name="tor_max">3.0</param>            <param name="direction">-1</param>            <command_interface name="effort" />
             <state_interface name="position" />
             <state_interface name="velocity" />
@@ -107,5 +111,6 @@
             <param name="offset">0</param>
             <param name="motor_type">M3508</param>
-            <command_interface name="effort" />
+            <param name="reduction">19.2032</param>
+            <param name="tor_max">3.0</param>            <param name="direction">1</param>            <command_interface name="effort" />
             <state_interface name="position" />
             <state_interface name="velocity" />
@@ -113,9 +118,10 @@
         <joint name="left_wheel_back_joint">
             <param name="motor_name">left_wheel_back_motor</param>
-            <param name="can_bus">can0</param>
-            <param name="tx_id">5</param>
+            <param name="can_bus">can1</param>
+            <param name="tx_id">4</param>
             <param name="offset">0</param>
             <param name="motor_type">M3508</param>
-            <command_interface name="effort" />
+            <param name="reduction">19.2032</param>
+            <param name="tor_max">3.0</param>            <param name="direction">-1</param>            <command_interface name="effort" />
             <state_interface name="position" />
             <state_interface name="velocity" />
@@ -124,8 +130,9 @@
             <param name="motor_name">right_wheel_back_motor</param>
             <param name="can_bus">can1</param>
-            <param name="tx_id">4</param>
+            <param name="tx_id">3</param>
             <param name="offset">0</param>
             <param name="motor_type">M3508</param>
-            <command_interface name="effort" />
+            <param name="reduction">19.2032</param>
+            <param name="tor_max">3.0</param>            <param name="direction">1</param>            <command_interface name="effort" />
             <state_interface name="position" />
             <state_interface name="velocity" />

File: src/spr_sentry_description/sentry.urdf.xacro (robot description, xacro)
@@ -73,5 +73,5 @@
   <link name="pitch_link">
     <visual>
-      <origin xyz="0.14 0 0" rpy="0 1.5708 0" />
+      <origin xyz="-0.14 0 0" rpy="0 1.5708 0" />
       <material name="">
         <color rgba="0 1 1 1" />
@@ -82,5 +82,5 @@
     </visual>
     <collision>
-      <origin xyz="0.14 0 0" rpy="0 1.5708 0" />
+      <origin xyz="-0.14 0 0" rpy="0 1.5708 0" />
       <geometry>
         <cylinder radius="0.05" length="0.28" />
@@ -112,5 +112,5 @@
   </link>
   <joint name="left_wheel_front_joint" type="continuous">
-    <origin xyz="-0.2 0.25 -0.05" rpy="0 0 0" />
+    <origin xyz="-0.2 -0.25 -0.05" rpy="0 0 0" />
     <parent link="base_link" />
     <child link="left_wheel_front_link" />
@@ -135,5 +135,5 @@
   </link>
   <joint name="right_wheel_front_joint" type="continuous">
-    <origin xyz="-0.2 -0.25 -0.05" rpy="0 0 0" />
+    <origin xyz="-0.2 0.25 -0.05" rpy="0 0 0" />
     <parent link="base_link" />
     <child link="right_wheel_front_link" />
@@ -158,5 +158,5 @@
     </link>
     <joint name="left_wheel_back_joint" type="continuous">
-      <origin xyz="0.2 0.25 -0.05" rpy="0 0 0" />
+      <origin xyz="0.2 -0.25 -0.05" rpy="0 0 0" />
       <parent link="base_link" />
       <child link="left_wheel_back_link" />
@@ -181,5 +181,5 @@
     </link>
     <joint name="right_wheel_back_joint" type="continuous">
-        <origin xyz="0.2 -0.25 -0.05" rpy="0 0 0" />
+        <origin xyz="0.2 0.25 -0.05" rpy="0 0 0" />
         <parent link="base_link" />
         <child link="right_wheel_back_link" />
